File: nrf51x22_qfax_dcdc.sch (KiCad schematic (older format))
At the start: 22 parts, among them U1 nrf51822-qfax, X1 Crystal-4, X2 32.768kHz

Commit message: WIP: Adding finished sch
Signed-off-by: Zamir SUN <sztsian@gmail.com>
Parts:
- removed C12: 1.0uF, dcdc:CAPC1608X06L, symbol C
- removed L4: 10uH, dcdc:INDC1608X06L, symbol L_Small
- removed L5: 15nH, dcdc:INDC1005X04L, symbol L_Small
- removed X1: Crystal-4, dcdc:BT-XTAL_2520, symbol Crystal-4
- added AE1: Antenna_Chip, RF_Antenna:Texas_SWRA117D_2.4GHz_Left, symbol Device:Antenna_Chip
- added J1: SWD, Connector_PinHeader_2.54mm:PinHeader_1x04_P2.54mm_Vertical, symbol Connector:Conn_01x04_Male
- added R1: 0R, Resistor_SMD:R_0402_1005Metric, symbol Device:R_Small
- added U2: nRF51822-WROOM-32, zsun-symbols:nRF51822-WROOM-32D, symbol zsun-lib:nRF51822-WROOM-32
- added Y1: 16M 3225, Crystal:Crystal_SMD_2520-4Pin_2.5x2.0mm, symbol Device:Crystal_GND24
- C1, C10, C11, C13, C14, C2, C3, C4, C5, C6, C8, C9: footprint dcdc:CAPC1005X04L -> Capacitor_SMD:C_0402_1005Metric; symbol C -> Device:C
- C7: footprint dcdc:CAPC1608X06L -> Capacitor_SMD:C_0402_1005Metric; symbol C -> Device:C
- L1, L2, L3: footprint dcdc:INDC1005X04L -> Inductor_SMD:L_0402_1005Metric; symbol L_Small -> Device:L_Small
- U1: symbol nrf51822-qfax -> nrf51x22_qfax_dcdc-rescue:nrf51822-qfax
- X2: footprint dcdc:XTAL_3215 -> Crystal:Crystal_SMD_3215-2Pin_3.2x1.5mm; symbol Crystal_Small -> nrf51x22_qfax_dcdc-rescue:Crystal_Small
Connections:
- net labels added: P0.00, P0.01, P0.02, P0.03, P0.04, P0.05, P0.06, P0.07, P0.08, P0.09, P0.10, P0.11, P0.12, P0.13, P0.14, P0.15, P0.16, P0.17, P0.18, P0.19, P0.20, P0.21, P0.22, P0.23, P0.24, P0.25, P0.28, P0.29, P0.30, SWCLK, SWDIO
- wire segments 57 -> 74
Other:
- note added: "ESP32-WROOM32 vs nRF51\nchip_pu = nRST/SWDIO\nNC = SWCLK\nIO16 RX = P0.11\nIO17 TX = P0.09"

Commit message: WIP: finish basic pcb. There are errors in gerber
Signed-off-by: Ziqian SUN(Zamir) <zsun@redhat.com>
Parts:
- added J2, J3: Conn_01x14_Male, Connector_PinHeader_1.27mm:PinHeader_1x14_P1.27mm_Vertical, symbol Connector:Conn_01x14_Male
- added J4: Conn_01x10_Male, Connector_PinHeader_1.27mm:PinHeader_1x10_P1.27mm_Vertical, symbol Connector:Conn_01x10_Male
- added U3: nRF51822-WROOM-32, zsun-symbols:nRF51822-WROOM-32D, symbol nrf51x22_qfax_dcdc-rescue:nRF51822-WROOM-32-zsun-lib
- U2: symbol zsun-lib:nRF51822-WROOM-32 -> nrf51x22_qfax_dcdc-rescue:nRF51822-WROOM-32-zsun-lib
Connections:
- net AVDD: now also J2.2 (Pin_2), U3.2 (VDD)
- net GND: now also J2.1 (Pin_1), J3.1 (Pin_1), J4.10 (Pin_10), U3.1 (GND), U3.15 (GND), U3.38 (GND)
- net P0.00: now also J2.6 (Pin_6), U3.6 (IO34)
- net P0.01: now also J2.7 (Pin_7), U3.7 (IO35)
- net P0.02: now also J2.8 (Pin_8), U3.8 (IO32)
- net P0.03: now also J2.9 (Pin_9), U3.9 (IO33)
- net P0.04: now also J2.10 (Pin_10), U3.10 (IO25)
- net P0.05: now also J2.11 (Pin_11), U3.11 (IO26)
- net P0.06: now also J2.12 (Pin_12), U3.12 (IO27)
- net P0.07: now also J2.13 (Pin_13), U3.13 (IO14)
- net P0.08: now also J2.14 (Pin_14), U3.14 (IO12)
- net P0.09: now also J3.11 (Pin_11), U3.28 (IO17)
- net P0.10: now also J4.9 (Pin_9), U3.16 (IO13)
- net P0.11: now also J3.12 (Pin_12), U3.27 (IO16)
- net P0.12: now also J4.8 (Pin_8), U3.17 (SHD/SD2)
- net P0.13: now also J4.7 (Pin_7), U3.18 (SWP/SD3)
- net P0.14: now also J4.6 (Pin_6), U3.19 (SCS/CMD)
- net P0.15: now also J4.5 (Pin_5), U3.20 (SCK/CLK)
- net P0.16: now also J4.4 (Pin_4), U3.21 (SDO/SD0)
- net P0.17: now also J4.3 (Pin_3), U3.22 (SDI/SD1)
- net P0.18: now also J4.2 (Pin_2), U3.23 (IO15)
- net P0.19: now also J4.1 (Pin_1), U3.24 (IO2)
- net P0.20: now also J3.14 (Pin_14), U3.25 (IO0)
- net P0.21: now also J3.13 (Pin_13), U3.26 (IO4)
- net P0.22: now also J3.10 (Pin_10), U3.29 (IO5)
- net P0.23: now also J3.9 (Pin_9), U3.30 (IO18)
- net P0.24: now also J3.8 (Pin_8), U3.31 (IO19)
- net P0.25: now also J3.6 (Pin_6), U3.33 (IO21)
- net P0.28: now also J3.5 (Pin_5), U3.34 (RXD0/IO3)
- net P0.29: now also J2.4 (Pin_4), U3.4 (SENSOR_VP)
- net P0.30: now also J2.5 (Pin_5), U3.5 (SENSOR_VN)
- net SWCLK: now also J3.7 (Pin_7), U3.32 (NC)
- net SWDIO: now also J2.3 (Pin_3), U3.3 (EN)
Other:
- moved on the sheet: J1, U2
